File: KiCAD_files/HATv1.0.kicad_pcb (KiCad board)
At the start: 4 copper layers, 65 x 56.5 mm, 43 parts, among them J1 Conn_Coaxial, J2 Conn_Coaxial, J3 USB_B_Micro, J4 raspberrypi_hat_OX40HAT, J5 Conn_01x04_Male, J6 Conn_01x06_Male, J7 Conn_01x02_Male, U1 mosaic-X5, U2 LD1117AS33TR, U3 SN74AVC4T245PW, U4 SN74LVC1G126DRLR

Commit message: Add files via upload
Parts:
- added G***: LOGO, openHW_small, F.Cu at (126.6, 71.8)
Changed lines of the file:
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@@
     (tracks 726)
     (zones 0)
-    (modules 43)
+    (modules 44)
     (nets 160)
   )
@@
     (add_net /USB_N)
     (add_net /USB_P)
+  )
+  (module openHW_small (layer F.Cu)
+    (at 126.61 71.83)
+    (fp_text reference G*** (at 0 0) (layer F.SilkS) hide
+      (effects (font (size 1.524 1.524) (thickness 0.3)))
+    )
+    (fp_text value LOGO (at 0.75 0) (layer F.SilkS) hide
+      (effects (font (size 1.524 1.524) (thickness 0.3)))
+    )
+    (fp_poly (pts (xy 0.265066 -1.26185) (xy 0.276859 -1.200908) (xy 0.288065 -1.146702) (xy 0.29796 -1.102455)
+      (xy 0.30582 -1.071389) (xy 0.31092 -1.056728) (xy 0.311303 -1.056233) (xy 0.323984 -1.049006)
+      (xy 0.351285 -1.036342) (xy 0.388835 -1.020029) (xy 0.432261 -1.001853) (xy 0.47719 -0.983601)
+      (xy 0.519251 -0.96706) (xy 0.554071 -0.954016) (xy 0.577278 -0.946256) (xy 0.58378 -0.94488)
+      (xy 0.595307 -0.950392) (xy 0.620686 -0.965721) (xy 0.657098 -0.989063) (xy 0.701728 -1.018611)
+      (xy 0.751758 -1.052561) (xy 0.752108 -1.052801) (xy 0.80244 -1.087143) (xy 0.847582 -1.117548)
+      (xy 0.884647 -1.142105) (xy 0.910751 -1.158902) (xy 0.922973 -1.166014) (xy 0.934142 -1.160834)
+      (xy 0.956473 -1.143415) (xy 0.987291 -1.116399) (xy 1.02392 -1.08243) (xy 1.063688 -1.04415)
+      (xy 1.103918 -1.004201) (xy 1.141937 -0.965226) (xy 1.17507 -0.929869) (xy 1.200643 -0.900772)
+      (xy 1.215981 -0.880577) (xy 1.2192 -0.873308) (xy 1.213685 -0.860173) (xy 1.198355 -0.833316)
+      (xy 1.175028 -0.795673) (xy 1.145522 -0.750181) (xy 1.11252 -0.701041) (xy 1.07879 -0.650967)
+      (xy 1.049447 -0.606158) (xy 1.026301 -0.569481) (xy 1.011163 -0.543801) (xy 1.00584 -0.532053)
+      (xy 1.00975 -0.518287) (xy 1.02027 -0.490271) (xy 1.035584 -0.452249) (xy 1.053876 -0.408462)
+      (xy 1.073329 -0.363152) (xy 1.092128 -0.32056) (xy 1.108455 -0.284929) (xy 1.120496 -0.260501)
+      (xy 1.125778 -0.251918) (xy 1.136864 -0.248446) (xy 1.164169 -0.241984) (xy 1.203943 -0.233284)
+      (xy 1.252432 -0.2231) (xy 1.305885 -0.212185) (xy 1.360549 -0.201292) (xy 1.412673 -0.191175)
+      (xy 1.458504 -0.182587) (xy 1.49429 -0.176281) (xy 1.516279 -0.173011) (xy 1.520249 -0.17272)
+      (xy 1.522377 -0.163174) (xy 1.523802 -0.13696) (xy 1.524581 -0.097716) (xy 1.524767 -0.049082)
+      (xy 1.524415 0.005305) (xy 1.523581 0.061807) (xy 1.522319 0.116784) (xy 1.520684 0.1666)
+      (xy 1.518732 0.207615) (xy 1.516517 0.236191) (xy 1.514094 0.24869) (xy 1.513881 0.248894)
+      (xy 1.501033 0.252712) (xy 1.471604 0.259458) (xy 1.429003 0.268412) (xy 1.37664 0.278855)
+      (xy 1.325166 0.288711) (xy 1.265846 0.300492) (xy 1.213591 0.312073) (xy 1.171788 0.32261)
+      (xy 1.143824 0.331263) (xy 1.13356 0.336397) (xy 1.125246 0.350708) (xy 1.111692 0.379661)
+      (xy 1.094639 0.418936) (xy 1.075829 0.464213) (xy 1.057001 0.511172) (xy 1.039899 0.555493)
+      (xy 1.026262 0.592857) (xy 1.017832 0.618942) (xy 1.015962 0.628157) (xy 1.021511 0.640561)
+      (xy 1.03688 0.666605) (xy 1.060188 0.703317) (xy 1.089555 0.747722) (xy 1.1176 0.788893)
+      (xy 1.150668 0.837762) (xy 1.179235 0.881777) (xy 1.201412 0.917878) (xy 1.215309 0.943006)
+      (xy 1.2192 0.953351) (xy 1.21235 0.964756) (xy 1.193587 0.9875) (xy 1.165588 1.01883)
+      (xy 1.131028 1.055994) (xy 1.092586 1.096239) (xy 1.052938 1.136811) (xy 1.014762 1.17496)
+      (xy 0.980733 1.207931) (xy 0.95353 1.232972) (xy 0.93583 1.24733) (xy 0.93102 1.24968)
+      (xy 0.920207 1.244196) (xy 0.895649 1.229014) (xy 0.860284 1.206032) (xy 0.817049 1.177153)
+      (xy 0.781389 1.152878) (xy 0.733449 1.120275) (xy 0.690484 1.091587) (xy 0.655651 1.068879)
+      (xy 0.632101 1.054213) (xy 0.623928 1.049804) (xy 0.607188 1.050962) (xy 0.578231 1.059937)
+      (xy 0.542735 1.074926) (xy 0.53848 1.07696) (xy 0.503347 1.092424) (xy 0.474165 1.102497)
+      (xy 0.456542 1.10529) (xy 0.45527 1.104974) (xy 0.449174 1.095097) (xy 0.43644 1.069051)
+      (xy 0.418184 1.029449) (xy 0.395526 0.978902) (xy 0.369583 0.920023) (xy 0.341475 0.855423)
+      (xy 0.312319 0.787715) (xy 0.283235 0.719512) (xy 0.255339 0.653424) (xy 0.229751 0.592065)
+      (xy 0.207589 0.538046) (xy 0.189972 0.493979) (xy 0.178018 0.462477) (xy 0.172844 0.446152)
+      (xy 0.17272 0.445044) (xy 0.180331 0.436594) (xy 0.200654 0.419375) (xy 0.229926 0.396509)
+      (xy 0.243447 0.386371) (xy 0.314254 0.322776) (xy 0.368154 0.250954) (xy 0.404981 0.173199)
+      (xy 0.42457 0.091801) (xy 0.426757 0.009053) (xy 0.411375 -0.072753) (xy 0.378259 -0.151324)
+      (xy 0.327245 -0.224368) (xy 0.290226 -0.262531) (xy 0.220158 -0.314645) (xy 0.144891 -0.34886)
+      (xy 0.066692 -0.366178) (xy -0.012173 -0.367598) (xy -0.089436 -0.35412) (xy -0.162831 -0.326746)
+      (xy -0.23009 -0.286475) (xy -0.288947 -0.234307) (xy -0.337135 -0.171243) (xy -0.372386 -0.098284)
+      (xy -0.392435 -0.016429) (xy -0.39624 0.040386) (xy -0.386636 0.131394) (xy -0.358018 0.215513)
+      (xy -0.310682 0.292185) (xy -0.244922 0.360854) (xy -0.212968 0.386371) (xy -0.181146 0.410632)
+      (xy -0.156751 0.430511) (xy -0.143546 0.442883) (xy -0.14224 0.445044) (xy -0.146106 0.458493)
+      (xy -0.156956 0.487569) (xy -0.173672 0.529662) (xy -0.195134 0.582158) (xy -0.220223 0.642446)
+      (xy -0.247819 0.707913) (xy -0.276803 0.775947) (xy -0.306056 0.843936) (xy -0.334458 0.909268)
+      (xy -0.360891 0.969331) (xy -0.384234 1.021512) (xy -0.403369 1.063199) (xy -0.417176 1.091781)
+      (xy -0.424536 1.104644) (xy -0.425071 1.105082) (xy -0.440478 1.103421) (xy -0.468385 1.094054)
+      (xy -0.503381 1.078873) (xy -0.51183 1.074775) (xy -0.5842 1.038946) (xy -0.738211 1.144313)
+      (xy -0.787593 1.177789) (xy -0.831368 1.206878) (xy -0.866731 1.229764) (xy -0.890881 1.244633)
+      (xy -0.900907 1.24968) (xy -0.910451 1.242806) (xy -0.931911 1.223657) (xy -0.962947 1.194439)
+      (xy -1.00122 1.157356) (xy -1.044393 1.114616) (xy -1.049157 1.109848) (xy -1.092419 1.065665)
+      (xy -1.130224 1.025454) (xy -1.160349 0.991713) (xy -1.18057 0.966939) (xy -1.188663 0.953629)
+      (xy -1.18872 0.953084) (xy -1.183164 0.93952) (xy -1.167756 0.912427) (xy -1.144384 0.874856)
+      (xy -1.114939 0.829862) (xy -1.08712 0.788893) (xy -1.05411 0.740315) (xy -1.025575 0.696928)
+      (xy -1.003396 0.661704) (xy -0.989454 0.637617) (xy -0.985483 0.628157) (xy -0.989254 0.612486)
+      (xy -0.999445 0.582527) (xy -1.014316 0.542599) (xy -1.032125 0.497023) (xy -1.051131 0.450117)
+      (xy -1.069593 0.406203) (xy -1.08577 0.369599) (xy -1.09792 0.344627) (xy -1.103081 0.336397)
+      (xy -1.117027 0.329943) (xy -1.147616 0.320906) (xy -1.191461 0.310129) (xy -1.245174 0.298454)
+      (xy -1.294687 0.288711) (xy -1.352823 0.277552) (xy -1.404198 0.267249) (xy -1.445404 0.258521)
+      (xy -1.473029 0.252087) (xy -1.483402 0.248894) (xy -1.485839 0.23793) (xy -1.488074 0.210579)
+      (xy -1.490051 0.170481) (xy -1.491715 0.121272) (xy -1.49301 0.066592) (xy -1.493883 0.010078)
+      (xy -1.494278 -0.04463) (xy -1.49414 -0.093895) (xy -1.493414 -0.134079) (xy -1.492046 -0.161542)
+      (xy -1.489979 -0.172647) (xy -1.48977 -0.17272) (xy -1.474037 -0.174633) (xy -1.443075 -0.179869)
+      (xy -1.400636 -0.187675) (xy -1.350472 -0.197297) (xy -1.296335 -0.207983) (xy -1.241977 -0.218978)
+      (xy -1.19115 -0.22953) (xy -1.147606 -0.238886) (xy -1.115098 -0.246291) (xy -1.097378 -0.250994)
+      (xy -1.095299 -0.251918) (xy -1.08792 -0.26452) (xy -1.074821 -0.29167) (xy -1.05782 -0.329126)
+      (xy -1.038732 -0.372645) (xy -1.019373 -0.417987) (xy -1.001559 -0.460909) (xy -0.987107 -0.49717)
+      (xy -0.977832 -0.522527) (xy -0.97536 -0.532053) (xy -0.980858 -0.544118) (xy -0.996142 -0.570001)
+      (xy -1.019404 -0.606835) (xy -1.048833 -0.651754) (xy -1.08204 -0.701041) (xy -1.115822 -0.75136)
+      (xy -1.145198 -0.796696) (xy -1.168352 -0.834111) (xy -1.183465 -0.860668) (xy -1.188721 -0.873308)
+      (xy -1.181808 -0.885995) (xy -1.162855 -0.909369) (xy -1.134535 -0.940789) (xy -1.099522 -0.97761)
+      (xy -1.060492 -1.01719) (xy -1.020119 -1.056887) (xy -0.981077 -1.094058) (xy -0.946041 -1.12606)
+      (xy -0.917685 -1.15025) (xy -0.898684 -1.163985) (xy -0.892494 -1.166014) (xy -0.880108 -1.1588)
+      (xy -0.853901 -1.14193) (xy -0.816757 -1.117317) (xy -0.771561 -1.086871) (xy -0.721629 -1.052801)
+      (xy -0.671572 -1.018828) (xy -0.626896 -0.989244) (xy -0.590419 -0.965854) (xy -0.564957 -0.950464)
+      (xy -0.553326 -0.944881) (xy -0.553301 -0.944881) (xy -0.539074 -0.94865) (xy -0.510634 -0.958766)
+      (xy -0.472353 -0.973442) (xy -0.428603 -0.990892) (xy -0.383756 -1.009329) (xy -0.342185 -1.026965)
+      (xy -0.308261 -1.042015) (xy -0.286358 -1.05269) (xy -0.280824 -1.056233) (xy -0.276095 -1.068763)
+      (xy -0.268521 -1.098075) (xy -0.258826 -1.140945) (xy -0.247736 -1.194152) (xy -0.235975 -1.254471)
+      (xy -0.234587 -1.26185) (xy -0.197857 -1.45796) (xy 0.228336 -1.45796) (xy 0.265066 -1.26185)) (layer F.SilkS) (width 0.01))
   )
   (module nice2 (layer B.Cu)
@@
     (pad U21 smd circle (at -6.35 11.43 180) (size 0.6 0.6) (layers F.Cu F.Paste F.Mask)
       (net 1 GND))
-    (model "C:/Users/JMA0162986/Documents/Github res/3d obj/mosaic3D.stp"
+    (model "C:/Users/JMA0162986/Documents/Github res/mosaic_design_components/mosaic3D.stp"
       (offset (xyz 15.5 -15.5 0))
       (scale (xyz 1 1 1))

Commit message: Add files via upload
Connections:
- U2 pad 4: +3V3 -> (no net)
